File: telescope/telescope/Buck.kicad_sch (KiCad schematic)
At the start: 4 parts

Commit message: Checkpoint for BLDC tracking mount controller
Parts:
- removed L_{buck}: 22uH, symbol Device:L_Small
- C_{buck}1: renamed from C2; footprint (none) -> Capacitor_SMD:C_0805_2012Metric
- LBK1: renamed from L_{buck}; footprint (none) -> Inductor_SMD:L_Bourns-SRN4018
- RBK1: renamed from R_{buck}; value R_Small -> 22R; footprint (none) -> Resistor_SMD:R_0805_2012Metric
Connections:
- net FB_{buck} renamed FBBK
- net GND_{buck} renamed GNDBK
- net SW_{buck} renamed SWBK
Other:
- moved on the sheet: C_{buck}1, LBK1, RBK1
Changed lines of the file:
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@@
 (kicad_sch (version 20230121) (generator eeschema)
   (paper "A4")
-  (junction (at 85.09 71.12) (diameter 0) (color 0 0 0 0)
+  (junction (at 88.9 78.74) (diameter 0) (color 0 0 0 0)
   )
   (junction (at 74.93 69.85) (diameter 0) (color 0 0 0 0)
   )
-  (junction (at 93.98 71.12) (diameter 0) (color 0 0 0 0)
+  (junction (at 93.98 69.85) (diameter 0) (color 0 0 0 0)
   )
   (junction (at 85.09 69.85) (diameter 0) (color 0 0 0 0)
   )
-  (junction (at 88.9 71.12) (diameter 0) (color 0 0 0 0)
+  (junction (at 88.9 69.85) (diameter 0) (color 0 0 0 0)
   )
-  (wire (pts (xy 74.93 77.47) (xy 77.47 77.47))
+  (wire (pts (xy 74.93 73.66) (xy 77.47 73.66))
     (stroke (width 0) (type default))
   )
@@
     (stroke (width 0) (type default))
   )
-  (wire (pts (xy 82.55 77.47) (xy 85.09 77.47))
+  (wire (pts (xy 82.55 73.66) (xy 85.09 73.66))
     (stroke (width 0) (type default))
   )
-  (wire (pts (xy 96.52 71.12) (xy 93.98 71.12))
+  (wire (pts (xy 96.52 69.85) (xy 93.98 69.85))
     (stroke (width 0) (type default))
   )
-  (wire (pts (xy 85.09 69.85) (xy 85.09 71.12))
+  (wire (pts (xy 85.09 69.85) (xy 85.09 73.66))
     (stroke (width 0) (type default))
   )
-  (wire (pts (xy 74.93 69.85) (xy 77.47 69.85))
+  (wire (pts (xy 85.09 67.31) (xy 85.09 69.85))
     (stroke (width 0) (type default))
   )
-  (wire (pts (xy 85.09 71.12) (xy 85.09 77.47))
+  (wire (pts (xy 96.52 67.31) (xy 93.98 67.31))
     (stroke (width 0) (type default))
   )
-  (wire (pts (xy 85.09 62.23) (xy 85.09 69.85))
+  (wire (pts (xy 77.47 67.31) (xy 74.93 67.31))
     (stroke (width 0) (type default))
   )
-  (wire (pts (xy 96.52 68.58) (xy 93.98 68.58))
+  (wire (pts (xy 74.93 67.31) (xy 74.93 69.85))
     (stroke (width 0) (type default))
   )
-  (wire (pts (xy 77.47 62.23) (xy 74.93 62.23))
+  (wire (pts (xy 82.55 67.31) (xy 85.09 67.31))
     (stroke (width 0) (type default))
   )
-  (wire (pts (xy 74.93 62.23) (xy 74.93 69.85))
+  (wire (pts (xy 88.9 69.85) (xy 85.09 69.85))
     (stroke (width 0) (type default))
   )
-  (wire (pts (xy 82.55 62.23) (xy 85.09 62.23))
+  (wire (pts (xy 74.93 69.85) (xy 74.93 73.66))
     (stroke (width 0) (type default))
   )
-  (wire (pts (xy 88.9 71.12) (xy 85.09 71.12))
+  (wire (pts (xy 96.52 78.74) (xy 88.9 78.74))
     (stroke (width 0) (type default))
   )
-  (wire (pts (xy 74.93 69.85) (xy 74.93 77.47))
+  (wire (pts (xy 93.98 69.85) (xy 88.9 69.85))
     (stroke (width 0) (type default))
   )
-  (wire (pts (xy 96.52 80.01) (xy 88.9 80.01))
+  (wire (pts (xy 88.9 69.85) (xy 88.9 71.12))
     (stroke (width 0) (type default))
   )
-  (wire (pts (xy 93.98 71.12) (xy 88.9 71.12))
+  (wire (pts (xy 93.98 67.31) (xy 93.98 69.85))
     (stroke (width 0) (type default))
   )
-  (wire (pts (xy 85.09 69.85) (xy 82.55 69.85))
+  (wire (pts (xy 88.9 76.2) (xy 88.9 78.74))
     (stroke (width 0) (type default))
   )
-  (wire (pts (xy 88.9 71.12) (xy 88.9 72.39))
-    (stroke (width 0) (type default))
-  )
-  (wire (pts (xy 93.98 68.58) (xy 93.98 71.12))
-    (stroke (width 0) (type default))
-  )
-  (wire (pts (xy 88.9 77.47) (xy 88.9 80.01))
-    (stroke (width 0) (type default))
-  )
-  (hierarchical_label "FB_{buck}" (shape input) (at 96.52 68.58 0) (fields_autoplaced)
+  (hierarchical_label "FBBK" (shape output) (at 96.52 67.31 0) (fields_autoplaced)
     (effects (font (size 1.27 1.27)) (justify left))
   )
-  (hierarchical_label "GND_{buck}" (shape output) (at 96.52 80.01 0) (fields_autoplaced)
+  (hierarchical_label "GNDBK" (shape output) (at 96.52 78.74 0) (fields_autoplaced)
     (effects (font (size 1.27 1.27)) (justify left))
   )
-  (hierarchical_label "V_{buck}" (shape output) (at 96.52 71.12 0) (fields_autoplaced)
+  (hierarchical_label "VBK" (shape output) (at 96.52 69.85 0) (fields_autoplaced)
     (effects (font (size 1.27 1.27)) (justify left))
   )
-  (hierarchical_label "SW_{buck}" (shape input) (at 63.5 69.85 180) (fields_autoplaced)
+  (hierarchical_label "SWBK" (shape input) (at 63.5 69.85 180) (fields_autoplaced)
     (effects (font (size 1.27 1.27)) (justify right))
   )
-  (symbol (lib_id "Device:L_Small") (at 80.01 69.85 90) (unit 1)
-    (in_bom yes) (on_board yes) (dnp yes) (fields_autoplaced)
-    (property "Reference" "L_{buck}" (at 80.01 64.77 90)
+  (symbol (lib_id "Device:L_Small") (at 80.01 67.31 90) (unit 1)
+    (in_bom yes) (on_board yes) (dnp no) (fields_autoplaced)
+    (property "Reference" "LBK1" (at 80.01 62.23 90)
       (effects (font (size 1.27 1.27)))
     )
-    (property "Value" "22uH" (at 80.01 67.31 90)
+    (property "Value" "47uH" (at 80.01 64.77 90)
       (effects (font (size 1.27 1.27)))
     )
-    (property "Footprint" "" (at 80.01 69.85 0)
+    (property "Footprint" "Inductor_SMD:L_Bourns-SRN4018" (at 80.01 67.31 0)
       (effects (font (size 1.27 1.27)) hide)
     )
-    (property "Datasheet" "~" (at 80.01 69.85 0)
-      (effects (font (size 1.27 1.27)) hide)
-    )
-    (property "Sim.Enable" "0" (at 80.01 69.85 0)
+    (property "Datasheet" "~" (at 80.01 67.31 0)
       (effects (font (size 1.27 1.27)) hide)
     )
@@
       (project "telescope"
         (path "/ab971623-295e-4b4e-9159-ef738a0d0f6a/a300b79c-df14-446a-a35d-0d329278ee79"
-          (reference "L_{buck}") (unit 1)
+          (reference "LBK1") (unit 1)
         )
       )
     )
   )
-  (symbol (lib_id "Device:L_Small") (at 80.01 62.23 90) (unit 1)
+  (symbol (lib_id "Device:C_Small") (at 88.9 73.66 0) (unit 1)
     (in_bom yes) (on_board yes) (dnp no) (fields_autoplaced)
-    (property "Reference" "L_{buck}" (at 80.01 57.15 90)
-      (effects (font (size 1.27 1.27)))
+    (property "Reference" "C_{buck}1" (at 91.44 72.3963 0)
+      (effects (font (size 1.27 1.27)) (justify left))
     )
-    (property "Value" "47uH" (at 80.01 59.69 90)
-      (effects (font (size 1.27 1.27)))
+    (property "Value" "10V 22uF" (at 91.44 74.9363 0)
+      (effects (font (size 1.27 1.27)) (justify left))
     )
-    (property "Footprint" "" (at 80.01 62.23 0)
+    (property "Footprint" "Capacitor_SMD:C_0805_2012Metric" (at 88.9 73.66 0)
       (effects (font (size 1.27 1.27)) hide)
     )
-    (property "Datasheet" "~" (at 80.01 62.23 0)
+    (property "Datasheet" "~" (at 88.9 73.66 0)
       (effects (font (size 1.27 1.27)) hide)
     )
@@
       (project "telescope"
         (path "/ab971623-295e-4b4e-9159-ef738a0d0f6a/a300b79c-df14-446a-a35d-0d329278ee79"
-          (reference "L_{buck}") (unit 1)
+          (reference "C_{buck}1") (unit 1)
         )
       )
     )
   )
-  (symbol (lib_id "Device:C_Small") (at 88.9 74.93 0) (unit 1)
-    (in_bom yes) (on_board yes) (dnp no) (fields_autoplaced)
-    (property "Reference" "C2" (at 91.44 73.6663 0)
-      (effects (font (size 1.27 1.27)) (justify left))
+  (symbol (lib_id "Device:R_Small") (at 80.01 73.66 90) (unit 1)
+    (in_bom yes) (on_board yes) (dnp yes)
+    (property "Reference" "RBK1" (at 80.01 76.2 90)
+      (effects (font (size 1.27 1.27)))
     )
-    (property "Value" "10V 22uF" (at 91.44 76.2063 0)
-      (effects (font (size 1.27 1.27)) (justify left))
+    (property "Value" "22R" (at 80.01 78.74 90)
+      (effects (font (size 1.27 1.27)))
     )
-    (property "Footprint" "" (at 88.9 74.93 0)
+    (property "Footprint" "Resistor_SMD:R_0805_2012Metric" (at 80.01 73.66 0)
       (effects (font (size 1.27 1.27)) hide)
     )
-    (property "Datasheet" "~" (at 88.9 74.93 0)
+    (property "Datasheet" "~" (at 80.01 73.66 0)
       (effects (font (size 1.27 1.27)) hide)
     )
@@
       (project "telescope"
         (path "/ab971623-295e-4b4e-9159-ef738a0d0f6a/a300b79c-df14-446a-a35d-0d329278ee79"
-          (reference "C2") (unit 1)
+          (reference "RBK1") (unit 1)
         )
       )
     )
   )
-  (symbol (lib_id "Device:R_Small") (at 80.01 77.47 90) (unit 1)
-    (in_bom yes) (on_board yes) (dnp yes) (fields_autoplaced)
-    (property "Reference" "R_{buck}" (at 80.01 72.39 90)
+  (symbol (lib_id "power:GND") (at 88.9 78.74 0) (unit 1)
+    (in_bom yes) (on_board yes) (dnp no) (fields_autoplaced)
+    (property "Reference" "#PWR011" (at 88.9 85.09 0)
+      (effects (font (size 1.27 1.27)) hide)
+    )
+    (property "Value" "BKGND" (at 88.9 83.82 0)
       (effects (font (size 1.27 1.27)))
     )
-    (property "Value" "R_Small" (at 80.01 74.93 90)
-      (effects (font (size 1.27 1.27)))
-    )
-    (property "Footprint" "" (at 80.01 77.47 0)
+    (property "Footprint" "" (at 88.9 78.74 0)
       (effects (font (size 1.27 1.27)) hide)
     )
-    (property "Datasheet" "~" (at 80.01 77.47 0)
+    (property "Datasheet" "" (at 88.9 78.74 0)
       (effects (font (size 1.27 1.27)) hide)
     )
     (pin "1")
-    (pin "2")
     (instances
       (project "telescope"
+        (path "/ab971623-295e-4b4e-9159-ef738a0d0f6a"
+          (reference "#PWR011") (unit 1)
+        )
         (path "/ab971623-295e-4b4e-9159-ef738a0d0f6a/a300b79c-df14-446a-a35d-0d329278ee79"
-          (reference "R_{buck}") (unit 1)
+          (reference "#PWR011") (unit 1)
         )
       )
