File: telescope/telescope/telescope.kicad_sch (KiCad schematic)
At the start: 21 parts, among them J1 V_{out}, J2 STEMMA QT, J3 OSTTC032162, U1 PMCF8316A1VRGFR

Commit message: Checkpoint for BLDC tracking mount controller
Parts:
- removed J1: V_{out}, symbol Connector:Conn_01x02_Pin
- removed J2: STEMMA QT, digikey-footprints:PinHeader_2x1mm_P2mm_SMD_RA, symbol dk_Rectangular-Connectors-Headers-Male-Pins:S2B-PH-SM4-TB_LF__SN_
- removed J3: OSTTC032162, digikey-footprints:TERM_BLOCK_1x3_P5.08MM, symbol dk_Terminal-Blocks-Wire-to-Board:OSTTC032162
- removed R7, R8: R_Small, symbol Device:R_Small
- added J1: Conn_01x03, TerminalBlock_Phoenix:TerminalBlock_Phoenix_MKDS-1,5-3-5.08_1x03_P5.08mm_Horizontal, symbol Connector_Generic:Conn_01x03
- added J2: STEMMA QT, Connector_JST:JST_PH_S2B-PH-K_1x02_P2.00mm_Horizontal, symbol Connector_Generic:Conn_01x02
- added NT1: NetTie_3, NetTie:NetTie-3_SMD_Pad2.0mm, symbol Device:NetTie_3
- added R9: 10K, Resistor_SMD:R_0805_2012Metric, symbol Device:R_Small
- added TPAVDD1, TPVDD1, TP_{EXT_WD}1, TP_{PGND}1, TP_{SPEED}2: 5000, TestPoint:TestPoint_Loop_D1.80mm_Drill1.0mm_Beaded, symbol Connector:TestPoint
- added TPBK1: TestPoint, TestPoint:TestPoint_Loop_D1.80mm_Drill1.0mm_Beaded, symbol Connector:TestPoint
- CAVDD1: renamed from C_{DVDD}1; footprint (none) -> Capacitor_SMD:C_0805_2012Metric; Specs (none) -> >=6.3V; 0.7µF > C > 1.3µF at 3.3V
- CCP1: renamed from C1; value 1uF, 16V X5R -> 1uF; footprint (none) -> Capacitor_SMD:C_0805_2012Metric; Specs (none) -> 16V X5R
- CDVDD1: renamed from C_{DVDD}; footprint (none) -> Capacitor_SMD:C_0805_2012Metric; Specs (none) -> X5R; >= 4V; 0.6µF > C > 1.3µF at 1.5V
- CFLY1: renamed from C2; value 47nF X5R -> 47nF; footprint (none) -> Capacitor_SMD:C_0805_2012Metric; Specs (none) -> X5R 24V
- CVM1: renamed from C4; footprint (none) -> Capacitor_SMD:C_0805_2012Metric; Specs (none) -> X5R 24V
- CVM2: renamed from C3; value 10uF X5R -> 100uF; footprint (none) -> Capacitor_SMD:C_1812_4532Metric; Specs (none) -> X5R 24V
- R1, R2, R3, R4, R5: footprint (none) -> Resistor_SMD:R_0805_2012Metric
- R6: value R_Small -> 10K; footprint (none) -> Resistor_SMD:R_0805_2012Metric
- TP_{FG}1: renamed from TP_{FG}; footprint digikey-footprints:Test_Point_D1.02mm -> TestPoint:TestPoint_Loop_D1.80mm_Drill1.0mm_Beaded; symbol dk_Test-Points:5000 -> Connector:TestPoint; now not fitted
- TP_{SOx}1: renamed from TP_{SOx}; footprint digikey-footprints:Test_Point_D1.02mm -> TestPoint:TestPoint_Loop_D1.80mm_Drill1.0mm_Beaded; symbol dk_Test-Points:5000 -> Connector:TestPoint; now not fitted
- TP_{nFAULT}1: renamed from TP_{nFAULT}; footprint digikey-footprints:Test_Point_D1.02mm -> TestPoint:TestPoint_Loop_D1.80mm_Drill1.0mm_Beaded; symbol dk_Test-Points:5000 -> Connector:TestPoint; now not fitted
- U1: footprint QFN_A1VRGFR_TEX -> Motor controller:QFN_A1VRGFR_TEX
Connections:
- net at R2.2, U1.30 (SDA): now also J2.2 (Pin_2)
- net at CDVDD1.2, U1.1 (DVDD): now also TPVDD1.1
- net at U1.13 (OUT_A), U1.14 (OUT_A): now also J1.1 (Pin_1)
- net at U1.16 (OUT_B), U1.17 (OUT_B): now also J1.2 (Pin_2)
- net at U1.19 (OUT_C), U1.20 (OUT_C): now also J1.3 (Pin_3)
- net at R1.2, U1.31 (SCL): now also J2.1 (Pin_1)
- net at U1.32 (EXT_WD): now also TP_{EXT_WD}1.1
- net TCXO/CLKOUT: now reaches U1.33 (EXT_CLK)
- net at U1.34 (DIR): now also R9.2
- net at U1.35 (BRAKE): now also R6.2
- net AV_{DD} renamed AVDD
- net AVDD: now also R9.1, TPAVDD1.1
- net Buck/FB_{buck} renamed Buck/FBBK
- net Buck/GND_{buck} renamed Buck/GNDBK
- net Buck/SW_{buck} renamed Buck/SWBK
- net GND renamed GNDA
- net GNDA: now also NT1.2; no longer U1.12 (PGND), U1.15 (PGND)
- net SPEED: no longer names the net of U1.28 (SPEED/WAKE)
- net SPEED: now also TP_{SPEED}2.1
- new net: NT1.1, TP_{PGND}1.1
- new net: U1.12 (PGND), U1.15 (PGND)
- new net Buck/VBK: TPBK1.1
Other:
- added sheet TCXO (TCXO.kicad_sch)
- sheet Buck ports: added FBBK, GNDBK, SWBK, VBK; removed FB_{buck}, GND_{buck}, SW_{buck}, V_{buck}
- moved on the sheet: CAVDD1, CCP1, CDVDD1, CFLY1, CVM1, CVM2, R1, R2, R3, R4, R5, R6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
